File: SAQ-Readout/SAQ-Readout.kicad_pcb (KiCad board)
At the start: 4 copper layers, 219.7 x 127 mm, 498 parts, among them J1 DB25_Female_MountingHoles, J3 Conn_01x06_Female, U1 IVC102, U10 AD8561, U11 IVC102, U12 AD8561, U13 IVC102, U14 AD8561, U15 IVC102, U16 AD8561, U17 IVC102, U18 AD8561, U19 IVC102, U2 AD8561, U20 AD8561, U21 IVC102, U22 AD8561, U23 IVC102, U24 AD8561, U25 IVC102, U26 AD8561, U27 IVC102, U28 AD8561, U29 IVC102, U3 IVC102, U30 AD8561, U31 IVC102, U32 AD8561, U4 AD8561, U5 IVC102, U6 AD8561, U7 IVC102, U8 AD8561, U9 IVC102

Commit message: Updated Readout
Parts:
- removed C10, C12, C13, C14, C15, C17, C18, C19, C20, C22, C23, C24, C25, C27, C28, C29, C30, C32, C33, C34, C35, C37, C38, C39, C40, C42, C43, C44, C45, C47, C48, C49, C50, C52, C53, C54, C55, C57, C58, C59, C60, C62, C63, C64, C65, C67, C68, C69, C7, C70, C72, C73, C74, C75, C77, C78, C79, C8, C80, C9: 0.1u, Capacitor_SMD:C_1206_3216Metric_Pad1.33x1.80mm_HandSolder
- removed C11, C16, C21, C26, C31, C36, C41, C46, C51, C56, C6, C61, C66, C71, C76: 10n, Capacitor_SMD:C_1206_3216Metric_Pad1.33x1.80mm_HandSolder
- removed J3: Conn_01x06_Female, Connector_TE-Connectivity:TE_MATE-N-LOK_1-770621-x_2x06_P4.14mm_Vertical
- removed R10, R16, R22, R28, R34, R40, R46, R52, R58, R64, R70, R76, R82, R88, R94: 2.2k, Resistor_SMD:R_0805_2012Metric_Pad1.20x1.40mm_HandSolder
- removed R11, R13, R17, R19, R23, R25, R29, R31, R35, R37, R41, R43, R47, R49, R53, R55, R59, R61, R65, R67, R7, R71, R73, R77, R79, R83, R85, R89, R91, R95: 50, Resistor_SMD:R_0805_2012Metric_Pad1.20x1.40mm_HandSolder
- removed R12, R15, R18, R21, R24, R27, R30, R33, R36, R39, R42, R45, R48, R51, R54, R57, R60, R63, R66, R69, R72, R75, R78, R81, R84, R87, R9, R90, R93, R96: 1k, Resistor_SMD:R_0805_2012Metric_Pad1.20x1.40mm_HandSolder
- removed R14, R20, R26, R32, R38, R44, R50, R56, R62, R68, R74, R8, R80, R86, R92: 3k, Resistor_SMD:R_0805_2012Metric_Pad1.20x1.40mm_HandSolder
- removed RV10, RV11, RV12, RV13, RV14, RV15, RV16, RV17, RV18, RV19, RV20, RV21, RV22, RV23, RV24, RV25, RV26, RV27, RV28, RV29, RV3, RV30, RV31, RV32, RV4, RV5, RV6, RV7, RV8, RV9: 0->10k, Potentiometer_SMD:Potentiometer_Bourns_3214W_Vertical
- removed TP1, TP10, TP11, TP12, TP13, TP14, TP15, TP16, TP3, TP4, TP5, TP6, TP7, TP8, TP9: TestPoint_Alt, TestPoint:TestPoint_THTPad_2.5x2.5mm_Drill1.2mm
- removed U10, U12, U14, U16, U18, U20, U22, U24, U26, U28, U30, U32, U4, U6, U8: AD8561, Package_SO:SOIC-8_3.9x4.9mm_P1.27mm
- removed U11, U13, U15, U17, U19, U21, U23, U25, U27, U29, U3, U31, U5, U7, U9: IVC102, Package_SO:SOIC-14_3.9x8.7mm_P1.27mm
- added G***: LOGO, LOGOs:UTA-LOGO-S0, F.Cu at (99.3, 34.0)
- added J2: Conn_02x06_Top_Bottom, Connector_TE-Connectivity:TE_MATE-N-LOK_1-770621-x_2x06_P4.14mm_Vertical, F.Cu at (229.7, 146.3)
- added REF**: MountingHole_3.2mm_M3, MountingHole:MountingHole_3.2mm_M3, F.Cu at (166.3, 117.4)
- added REF**: TestPoint_Pad_D2.0mm, TestPoint:TestPoint_Pad_D2.0mm, B.Cu at (136.9, 89.8)
- added REF**: TestPoint_Pad_D2.0mm, TestPoint:TestPoint_Pad_D2.0mm, B.Cu at (89.3, 89.8)
- added REF**: TestPoint_Pad_D2.0mm, TestPoint:TestPoint_Pad_D2.0mm, B.Cu at (113.1, 89.8)
- added REF**: TestPoint_Pad_D2.0mm, TestPoint:TestPoint_Pad_D2.0mm, B.Cu at (160.2, 76.0)
- added REF**: TestPoint_Pad_D2.0mm, TestPoint:TestPoint_Pad_D2.0mm, B.Cu at (65.4, 89.8)
- added REF**: TestPoint_Pad_D2.0mm, TestPoint:TestPoint_Pad_D2.0mm, B.Cu at (88.6, 76.0)
- added REF**: TestPoint_Pad_D2.0mm, TestPoint:TestPoint_Pad_D2.0mm, B.Cu at (208.5, 89.8)
- added REF**: TestPoint_Pad_D2.0mm, TestPoint:TestPoint_Pad_D2.0mm, B.Cu at (207.8, 75.9)
- added REF**: TestPoint_Pad_D2.0mm, TestPoint:TestPoint_Pad_D2.0mm, B.Cu at (136.3, 76.0)
- added REF**: TestPoint_Pad_D2.0mm, TestPoint:TestPoint_Pad_D2.0mm, B.Cu at (160.8, 89.8)
- added REF**: MountingHole_3.2mm_M3, MountingHole:MountingHole_3.2mm_M3, F.Cu at (218.1, 146.8)
- added REF**: TestPoint_Pad_D2.0mm, TestPoint:TestPoint_Pad_D2.0mm, B.Cu at (184.0, 76.0)
- added REF**: TestPoint_Pad_D2.0mm, TestPoint:TestPoint_Pad_D2.0mm, B.Cu at (298.7, 64.2)
- added REF**: TestPoint_Pad_D2.0mm, TestPoint:TestPoint_Pad_D2.0mm, B.Cu at (184.7, 89.8)
- added REF**: MountingHole_3.2mm_M3, MountingHole:MountingHole_3.2mm_M3, F.Cu at (243.1, 30.5)
- added REF**: MountingHole_3.2mm_M3, MountingHole:MountingHole_3.2mm_M3, F.Cu at (50.1, 30.5)
- added REF**: MountingHole_3.2mm_M3, MountingHole:MountingHole_3.2mm_M3, F.Cu at (50.1, 147.3)
- added REF**: TestPoint_Pad_D2.0mm, TestPoint:TestPoint_Pad_D2.0mm, B.Cu at (232.4, 89.7)
- added REF**: TestPoint_Pad_D2.0mm, TestPoint:TestPoint_Pad_D2.0mm, B.Cu at (231.7, 76.0)
- added REF**: TestPoint_Pad_D2.0mm, TestPoint:TestPoint_Pad_D2.0mm, B.Cu at (112.5, 76.0)
- added REF**: TestPoint_Pad_D2.0mm, TestPoint:TestPoint_Pad_D2.0mm, B.Cu at (64.8, 76.0)
Routing:
- net CH15: track 0.00 -> 188.0 mm
- net CH2: track 1611.5 -> 1518.2 mm
- net +15V: track 471.7 -> 538.8 mm
- net -15V: track 532.9 -> 598.6 mm
- net +5V: track 505.8 -> 569.6 mm
- net +9V: track 543.4 -> 601.5 mm
- net CH12: track 56.5 -> 0.00 mm
- net CH6: track 38.2 -> 0.00 mm
- net GND: track 1751.8 -> 1760.1 mm
Other:
- board text added: "+15V"
- board text added: "+5V"
- board text added: "+9V"
- board text added: "-15V"
- board text added: "Austin McDonald James Battat Joanthan Asaadi"
- board text added: "GND"
- board text added: "GNDD"
- board text added: "SAQ 16 Channel readout Aug 12th 2022"
