File: SAQ-Readout/SAQ-Readout.kicad_sch (KiCad schematic)
At the start: 3 parts, among them J1 DB25_Female_MountingHoles, J2 Conn_01x04_Female, J3 Conn_01x06_Female

Commit message: Updated Readout
Parts:
- removed J2: Conn_01x04_Female, symbol Connector:Conn_01x04_Female
- removed J3: Conn_01x06_Female, Connector_TE-Connectivity:TE_MATE-N-LOK_1-770621-x_2x06_P4.14mm_Vertical, symbol Connector:Conn_01x06_Female
- added J2: Conn_02x06_Top_Bottom, Connector_TE-Connectivity:TE_MATE-N-LOK_1-770621-x_2x06_P4.14mm_Vertical, symbol Connector_Generic:Conn_02x06_Top_Bottom
Connections:
- net GND: now also J2.1 (Pin_1), J2.2 (Pin_2), J2.7 (Pin_7), J2.8 (Pin_8)
- new net +15V: J2.12 (Pin_12), J2.6 (Pin_6)
- new net +5V: J2.10 (Pin_10), J2.4 (Pin_4)
- new net +9V: J2.3 (Pin_3), J2.9 (Pin_9)
- new net -15V: J2.11 (Pin_11), J2.5 (Pin_5)
